Commit message: Arm location changed to the middle of the plate

File: multirobot_description/urdf/mobile_ur10e.xacro (robot description, xacro)
@@ -21,5 +21,5 @@
     <update_rate>1</update_rate>
   <!-- Include UR10e Arm -->
-  <xacro:property name="arm_position_x" value="0.45"/>
+  <xacro:property name="arm_position_x" value="0.42"/>
   <xacro:property name="arm_position_y" value="0"/>
   <xacro:property name="arm_position_z" value="0"/>

Commit message: New URDF file design for both 'caster' and '4wd' mobile platform

File: multirobot_description/urdf/mobile_ur10e.xacro (robot description, xacro)
@@ -3,4 +3,5 @@
   <xacro:arg name="wheel_kind" default="default" /> <!-- default | tractor | tractor_large -->
   <xacro:arg name="front_kind" default="4wd" /> <!-- swing_axle | caster | 4wd -->
+  <xacro:property name="wheel_type" value='$(arg front_kind)'/>
   <!-- heros base-->
   <xacro:include filename="$(find innok_heros_description)/urdf/innok_heros_universal.xacro"/>
@@ -11,4 +12,5 @@
   <!-- ROS plug-ins -->
   <xacro:include filename="$(find multirobot_description)/urdf/ROS/mobile_arm_joint_pub.xacro" />
+  <xacro:include filename="$(find multirobot_description)/urdf/ROS/mobile_arm_joint_caster_pub.xacro" />
   <!-- Internal Measurement Unit -->
   <xacro:include filename="$(find multirobot_description)/urdf/sensors/internal_measurement_unit.urdf.xacro"/>
@@ -21,5 +23,10 @@
     <update_rate>1</update_rate>
   <!-- Include UR10e Arm -->
-  <xacro:property name="arm_position_x" value="0.42"/>
+  <xacro:if value="${wheel_type == '4wd'}">
+    <xacro:property name="arm_position_x" value="0.42"/>
+  </xacro:if>
+  <xacro:unless value="${wheel_type == '4wd'}">
+    <xacro:property name="arm_position_x" value="0.101"/>
+  </xacro:unless>
   <xacro:property name="arm_position_y" value="0"/>
   <xacro:property name="arm_position_z" value="0"/>
@@ -47,5 +54,10 @@
   </xacro:macro>
   <xacro:multirobot_mobile prefix="$(arg prefix)"/>
-  <xacro:mobile_arm_joint_pub/>
+  <xacro:if value="${wheel_type == '4wd'}">
+    <xacro:mobile_arm_joint_pub/>
+  </xacro:if>
+  <xacro:unless value="${wheel_type == '4wd'}">
+    <xacro:mobile_arm_joint_caster_pub/>
+  </xacro:unless>
   <!-- <xacro:mobile_arm_ros_control/> -->
 </robot>
